File: UglyFace_03.kicad_pcb (KiCad board)
At the start: 2 copper layers, 53 x 52.1 mm, 54 parts, among them J1 9V, J2 9V GND, J3 IN, J4 IN GND, J5 OUT, J6 OUT GND, J7 LED -, J8 LED GND, U1 TL072, U2 TLC555, U3 Vactrol

Commit message: Ugly Face 3 v1.1: C4 100u, RESET 22k, filtered 555 supply, clean dry path, buffered VB, THRESHOLD toggle, GLITCH trimmer, D3/D4 LED pads
As ordered from JLCPCB (October 2026 batch).

Co-Authored-By: Claude Opus 5.5 <noreply@anthropic.com>
Parts:
- added C17: 4.7u, Capacitor_SMD:C_0805_2012Metric_Pad1.18x1.45mm_HandSolder, F.Cu at (155.8, 122.6)
- added C18: 22u, Capacitor_SMD:C_1206_3216Metric_Pad1.33x1.80mm_HandSolder, F.Cu at (154.0, 113.0)
- added C19: 100n, Capacitor_SMD:C_0805_2012Metric_Pad1.18x1.45mm_HandSolder, F.Cu at (152.0, 115.4)
- added D3: 1N4148/LED, UglyFace:D_THT_Standing_3mm_P2.54_Compact, F.Cu at (141.7, 118.3)
- added D4: 1N4148/LED, UglyFace:D_THT_Standing_3mm_P2.54_Compact, F.Cu at (144.2, 122.8)
- added R20: 1k, Resistor_SMD:R_0805_2012Metric_Pad1.20x1.40mm_HandSolder, F.Cu at (123.9, 125.5)
- added R21: 2k2, Resistor_SMD:R_0805_2012Metric_Pad1.20x1.40mm_HandSolder, F.Cu at (126.4, 125.5)
- added R22: 22k, Resistor_SMD:R_0805_2012Metric_Pad1.20x1.40mm_HandSolder, F.Cu at (128.9, 125.5)
- added R23: 47, Resistor_SMD:R_0805_2012Metric_Pad1.20x1.40mm_HandSolder, F.Cu at (153.3, 110.5)
- added R24: 33k, Resistor_SMD:R_0805_2012Metric_Pad1.20x1.40mm_HandSolder, F.Cu at (152.0, 125.4)
- added R25: 10k, Resistor_SMD:R_0805_2012Metric_Pad1.20x1.40mm_HandSolder, F.Cu at (155.8, 118.5)
- added SW1: THR, UglyFace:SW_Taiway_100_SPDT_PC, B.Cu at (130.9, 110.1)
- added U4: TL072, Package_SO:SOIC-8_3.9x4.9mm_P1.27mm, F.Cu at (152.0, 120.3)
- C12, C13: value 100n -> 1u
- C4: value 22u -> 100u; footprint Capacitor_SMD:C_1206_3216Metric_Pad1.33x1.80mm_HandSolder -> Capacitor_SMD:CP_Elec_6.3x7.7
- C7: value 10u -> 2.2u
- R13: value 15k -> 47k
- RV2: value B10k -> 10k; footprint UglyFace:Potentiometer_Alpha_16mm_Vertical -> UglyFace:Potentiometer_Bourns_3362P_Vertical
- moved R19 36.3 mm to (157.0, 83.4), turned to 0 degrees
- moved R9 16.8 mm to (139.6, 121.0), turned to 90 degrees
- moved R5 5.99 mm to (135.3, 106.5), turned to 0 degrees
- moved R6 5.15 mm to (136.0, 114.5), turned to 0 degrees
- moved RV2 3.77 mm to (134.5, 123.6), turned to 180 degrees
- moved R4 3.55 mm to (128.5, 102.0), turned to 0 degrees
- moved C15 2.35 mm to (158.0, 120.9)
Connections:
- net Net-(U1A-+) renamed /PRE_IN
- C13 pad 1: /PRE_OUT -> /DRY_OUT
- C3 pad 1: +9V -> /V555
- C4 pad 1: /VB -> /VB_RAW
- C9 pad 2: /RESET -> /GATE_BIAS
- R1 pad 2: /VB -> /VB_RAW
- R2 pad 1: /VB -> /VB_RAW
- RV2 pad 2: /RESET -> /GATE_BIAS
- U2 pad 8: +9V -> /V555
Routing:
- net GND: track 167.2 -> 254.2 mm, vias 9 -> 2
- net /DRY_OUT: track 0.00 -> 57.0 mm, vias 0 -> 1
- net /VB: track 55.5 -> 91.8 mm, vias 3 -> 2
- net /VB_RAW: track 0.00 -> 32.5 mm, vias 0 -> 2
- net +9V: track 121.7 -> 153.9 mm, vias 2 -> 3
- net Net-(D3-K): track 0.00 -> 29.7 mm
- net /GATE_BIAS: track 0.00 -> 29.4 mm
- net Net-(SW1-A): track 0.00 -> 24.0 mm
- net Net-(R9-Pad1): track 26.5 -> 2.95 mm
- net /PRE_IN: track 18.7 -> 39.7 mm
- net Net-(D2-A): track 11.0 -> 31.7 mm
- net /V555: track 0.00 -> 19.6 mm
- net Net-(R12-Pad2): track 14.5 -> 27.5 mm
- net /RESET: track 46.1 -> 34.4 mm, vias 1 -> 2
- net Net-(SW1-C): track 0.00 -> 11.6 mm
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Other:
- board text added: "Deformis v3"
- board text removed: "Deformis v2"

Commit message: UF3 v1.3 PCB: new envelope parts placed and routed, slotted Taiway footprint, R31/R32 Basic 100k; renders, schematic PDF, docs
Board synced to schematic rev 1.3 (U5, Q1, D5, D6, C20-C22, R26-R36, RV6 added; R7, C8 removed; R13 220k, R21 15k, RV1 A10k).
Fully routed (46 vias), DRC 0 errors, parity clean. Envelope not breadboarded yet.

Co-Authored-By: Claude Opus 5.5 <noreply@anthropic.com>
Parts:
- removed C8: 100u, Capacitor_SMD:CP_Elec_6.3x7.7
- removed R7: 100, Resistor_SMD:R_0805_2012Metric_Pad1.20x1.40mm_HandSolder
- added C20: 33n, Capacitor_SMD:C_0805_2012Metric_Pad1.18x1.45mm_HandSolder, F.Cu at (146.7, 118.7)
- added C21: 1u, Capacitor_SMD:C_0805_2012Metric_Pad1.18x1.45mm_HandSolder, F.Cu at (162.2, 120.7)
- added C22: 100n, Capacitor_SMD:C_0805_2012Metric_Pad1.18x1.45mm_HandSolder, F.Cu at (167.0, 104.0)
- added D5: 1N4148W, Diode_SMD:D_SOD-123, F.Cu at (169.2, 113.4)
- added D6: BAT54S, Package_TO_SOT_SMD:SOT-23, F.Cu at (158.7, 112.9)
- added Q1: MMBT3904, Package_TO_SOT_SMD:SOT-23, F.Cu at (164.2, 112.9)
- added R26: 10k, Resistor_SMD:R_0805_2012Metric_Pad1.20x1.40mm_HandSolder, F.Cu at (158.2, 125.2)
- added R27: 1k, Resistor_SMD:R_0805_2012Metric_Pad1.20x1.40mm_HandSolder, F.Cu at (168.2, 120.9)
- added R28: 470k, Resistor_SMD:R_0805_2012Metric_Pad1.20x1.40mm_HandSolder, F.Cu at (166.0, 115.9)
- added R29: 22k, Resistor_SMD:R_0805_2012Metric_Pad1.20x1.40mm_HandSolder, F.Cu at (165.2, 118.9)
- added R30: 22k, Resistor_SMD:R_0805_2012Metric_Pad1.20x1.40mm_HandSolder, F.Cu at (160.5, 86.4)
- added R31: 100k, Resistor_SMD:R_0805_2012Metric_Pad1.20x1.40mm_HandSolder, F.Cu at (172.2, 118.9)
- added R32: 100k, Resistor_SMD:R_0805_2012Metric_Pad1.20x1.40mm_HandSolder, F.Cu at (168.2, 118.9)
- added R33: 1k, Resistor_SMD:R_0805_2012Metric_Pad1.20x1.40mm_HandSolder, F.Cu at (170.0, 116.9)
- added R34: 330, Resistor_SMD:R_0805_2012Metric_Pad1.20x1.40mm_HandSolder, F.Cu at (167.0, 112.9)
- added R35: 100, Resistor_SMD:R_0805_2012Metric_Pad1.20x1.40mm_HandSolder, F.Cu at (153.7, 83.9)
- added R36: 1M, Resistor_SMD:R_0805_2012Metric_Pad1.20x1.40mm_HandSolder, F.Cu at (172.2, 120.9)
- added RV6: 500k, UglyFace:Potentiometer_Bourns_3362P_Vertical, F.Cu at (165.5, 84.4)
- added U5: LM358, Package_SO:SOIC-8_3.9x4.9mm_P1.27mm, F.Cu at (167.0, 108.0)
- R13: value 47k -> 220k
- R21: value 2k2 -> 15k
- RV1: value B1k -> A10k
Connections:
- RV1 pad 1: GND -> /VB
- RV1 pad 2: /VACT_LED -> Net-(U5A-+)
- U3 pad 1: /VACT_LED -> Net-(U3-A)
- U3 pad 2: GND -> Net-(Q1-C)
Routing:
- net /ENV: track 0.00 -> 46.5 mm, vias 0 -> 4
- net /VACT_LED: track 40.7 -> 0.00 mm
- net /PRE_OUT: track 57.8 -> 19.0 mm
- net +9V: track 153.9 -> 189.2 mm, vias 3 -> 7
- net /VB: track 91.8 -> 121.4 mm, vias 2 -> 3
- net Net-(Q1-C): track 0.00 -> 24.9 mm, vias 0 -> 1
- net GND: track 254.2 -> 232.9 mm, vias 2 -> 3
- net Net-(U5A-+): track 0.00 -> 17.1 mm, vias 0 -> 1
- net /RESET: track 34.4 -> 50.4 mm
- net Net-(U5B--): track 0.00 -> 15.9 mm
- net Net-(Q1-B): track 0.00 -> 14.7 mm
- net /IN: track 42.6 -> 56.6 mm
- net Net-(C20-Pad2): track 0.00 -> 13.8 mm, vias 0 -> 2
- net Net-(R12-Pad2): track 27.5 -> 14.5 mm
- net Net-(R33-Pad1): track 0.00 -> 12.7 mm
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
Commit message: v1.3 = FU-2: silk 'FU-2 v1.3', R8 47k (Basic), C21 4.7u (bench-tested envelope), schematic title; envelope breadboard sheet; docs, renders
Co-Authored-By: Claude Opus 5.5 <noreply@anthropic.com>
Parts:
- C21: value 1u -> 4.7u
- R8: value 56k -> 47k
Other:
- board text added: "FU-2 v1.3"
- board text removed: "Deformis v3"
Changed lines of the file:
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@@
 			)
 		)
-		(property "Value" "56k"
+		(property "Value" "47k"
 			(at 0 1.65 0)
 			(layer "F.Fab")
@@
 			)
 		)
-		(property "Description" "Threshold top"
+		(property "Description" "Threshold top (v1.3: 47k, was 56k; JLC Basic. GLITCH range at RV2 ~0.15-1.66 V, trim point ~60%)"
 			(at 0 0 0)
 			(layer "F.Fab")
@@
 			)
 		)
-		(property "LCSC" "C17756"
+		(property "LCSC" "C17713"
 			(at 0 0 0)
 			(layer "F.SilkS")
@@
 			)
 		)
-		(property "Value" "1u"
+		(property "Value" "4.7u"
 			(at 0 1.68 180)
 			(layer "F.Fab")
@@
 			)
 		)
-		(property "Description" "Envelope hold cap"
+		(property "Description" "Envelope hold cap: 4.7u 25V X5R (~3u at the 4.5-7 V DC bias; bench-tested 3.3u film-equivalent on unit 1, 2026-10-23)"
 			(at 0 0 180)
 			(layer "F.Fab")
@@
 			)
 		)
-		(property "LCSC" "C28323"
+		(property "LCSC" "C1779"
 			(at 0 0 0)
 			(layer "F.Fab")
@@
 		)
 	)
-	(gr_text "Deformis v3"
+	(gr_text "FU-2 v1.3"
 		(at 123.25 130 0)
 		(layer "F.SilkS")
